File: Designs/Ionto_Current_Source_Core/variants/Ionto_Current_Source_Core_With_Pour.kicad_pcb (KiCad board)
At the start: 2 copper layers, 27 x 20 mm, 8 parts, among them J1 BATTERY INPUT 3.0-4.2V, J2 STIM OUTPUT, J3 CE JUMPER: 1=VIN 2=CE, U1 R1218N041A-TR-FE

Commit message: feat: optimize pcb manufacturing variants and previews
Routing:
- added copper zone on F.Cu, net GND
Changed lines of the file:
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@@
 	)
 	(embedded_fonts no)
+	(zone
+		(net "GND")
+		(layer "F.Cu")
+		(name "GND_TOP")
+		(hatch edge 0.508)
+		(connect_pads
+			(clearance 1)
+		)
+		(min_thickness 0.25)
+		(fill yes
+			(thermal_gap 0.5)
+			(thermal_bridge_width 0.5)
+			(island_removal_mode 0)
+		)
+		(polygon
+			(pts
+				(xy 21 21)
+				(xy 46 21)
+				(xy 46 39)
+				(xy 21 39)
+			)
+		)
+	)
 )
